File: Electronics/LED-shield/Direct-drive-LEDs/Direct-drive-LEDs.sch (KiCad schematic (older format))
At the start: 16 parts, among them J1 Conn_01x05_Female, J2 Conn_01x02_Female, J3 Conn_01x02_Male, Q1 MMBT3904, Q2 BS170F, Q3 Q_Photo_NPN, U1 TLC2272

Commit message: PCB for 4 LEDs.
Parts:
- removed C1: 100nF, Capacitor_SMD:C_0805_2012Metric_Pad1.15x1.40mm_HandSolder, symbol Device:C
- removed J1: Conn_01x05_Female, symbol Connector:Conn_01x05_Female
- removed J3: Conn_01x02_Male, symbol Connector:Conn_01x02_Male
- removed Q3: Q_Photo_NPN, symbol Device:Q_Photo_NPN
- removed R3: 3K3, Resistor_SMD:R_0805_2012Metric, symbol Device:R
- removed U1: TLC2272, Package_SO:SOIC-8-N7_3.9x4.9mm_P1.27mm, symbol Amplifier_Operational:OPA2277
- added C2, C6: 100nF, Capacitor_SMD:C_0805_2012Metric_Pad1.15x1.40mm_HandSolder, symbol Device:C
- added C3, C4, C5: 220nF, Capacitor_SMD:C_0805_2012Metric_Pad1.15x1.40mm_HandSolder, symbol Device:C
- added J1: Conn_01x11_Male, Connector_PinHeader_2.54mm:PinHeader_1x11_P2.54mm_Vertical, symbol Connector:Conn_01x11_Male
- added LED2, LED3, LED4: LED3MM, LED_THT:LED_D3.0mm, symbol adafruit-new:LED3MM
- added Q3, Q5, Q7: MMBT3904, Package_TO_SOT_SMD:SOT-23, symbol Transistor_BJT:MMBT3904
- added Q4, Q6, Q8: BS170F, Package_TO_SOT_SMD:SOT-23, symbol Transistor_FET:BS170F
- added R10, R18, R19: 10K, Resistor_SMD:R_0805_2012Metric, symbol Device:R
- added R11, R20, R21: 100R, Resistor_SMD:R_0805_2012Metric, symbol Device:R
- added R12, R13, R7: 33K, Resistor_SMD:R_0805_2012Metric, symbol Device:R
- added R14, R15, R8: 120K, Resistor_SMD:R_0805_2012Metric, symbol Device:R
- added R16, R17, R9: 330K, Resistor_SMD:R_0805_2012Metric, symbol Device:R
- added R5: 3K3, Resistor_SMD:R_0805_2012Metric, symbol Device:R
- added U1, U2: OP275, Package_SO:SOIC-8_3.9x4.9mm_P1.27mm, symbol Amplifier_Operational:OP275
- J2: footprint (none) -> Connector_PinHeader_2.54mm:PinHeader_1x02_P2.54mm_Vertical
- LED1: footprint adafruit-new_LED3MM -> LED_THT:LED_D3.0mm
- renumbered C2 to C1, R4 to R3, R5 to R4
Connections:
- net labels added: LEDon0, LEDon1, LEDon2, LEDon3, PWMin0, PWMin1, PWMin2, PWMin3
- net labels removed: LEDon, PWMin, Vout
- wire segments 48 -> 128
Other:
- moved on the sheet: C1, Q1, Q2, R1, R2, R3, R4, R6

Commit message: Arduino MEGA shield for half-neuron WIP.
Parts:
- removed J1: Conn_01x11_Male, Connector_PinHeader_2.54mm:PinHeader_1x11_P2.54mm_Vertical, symbol Connector:Conn_01x11_Male
- removed J2: Conn_01x02_Female, Connector_PinHeader_2.54mm:PinHeader_1x02_P2.54mm_Vertical, symbol Connector:Conn_01x02_Female
- removed LED1, LED2, LED3, LED4: LED3MM, LED_THT:LED_D3.0mm, symbol adafruit-new:LED3MM
- added D1, D2, D3, D4: LED, LED_THT:LED_D3.0mm, symbol Device:LED
- added XA1: Arduino_Mega2560_Shield, arduino:Arduino_Mega2560_Shield, symbol arduino:Arduino_Mega2560_Shield
Connections:
- net labels added: PhotoE, photoC
- wire segments 128 -> 135
Other:
- moved on the sheet: C2, C6, R5

Commit message: Minor PCB mods WIP.
Parts:
- added H1, H2: MountingHole, MountingHole:MountingHole_2.1mm, symbol Mechanical:MountingHole
- added J1: Conn_01x02_Male, Connector_PinHeader_2.54mm:PinHeader_1x02_P2.54mm_Vertical, symbol Connector:Conn_01x02_Male
Connections:
- net GND: now also J1.1 (Pin_1)
- net photoC: now also J1.2 (Pin_2)
Changed lines of the file:
@@
 Text GLabel 1750 6775 2    50   Input ~ 0
 photoC
-Text GLabel 1750 7050 2    50   Input ~ 0
-PhotoE
 Wire Wire Line
 	1750 6775 1625 6775
@@
 Wire Wire Line
 	5550 6525 5550 6325
+$Comp
+L Connector:Conn_01x02_Male J1
+U 1 1 5FF245E8
+P 1950 7050
+F 0 "J1" H 1922 6932 50  0000 R CNN
+F 1 "Conn_01x02_Male" H 1922 7023 50  0000 R CNN
+F 2 "Connector_PinHeader_2.54mm:PinHeader_1x02_P2.54mm_Vertical" H 1950 7050 50  0001 C CNN
+F 3 "~" H 1950 7050 50  0001 C CNN
+	1    1950 7050
+	-1   0    0    1
+$EndComp
+Wire Wire Line
+	1750 6950 1625 6950
+Wire Wire Line
+	1625 6950 1625 6775
+Connection ~ 1625 6775
+$Comp
+L Mechanical:MountingHole H2
+U 1 1 5FF32EFD
+P 4550 7375
+F 0 "H2" H 4650 7421 50  0000 L CNN
+F 1 "MountingHole" H 4650 7330 50  0000 L CNN
+F 2 "MountingHole:MountingHole_2.1mm" H 4550 7375 50  0001 C CNN
+F 3 "~" H 4550 7375 50  0001 C CNN
+	1    4550 7375
+	1    0    0    -1
+$EndComp
+$Comp
+L Mechanical:MountingHole H1
+U 1 1 5FF38966
+P 4300 7375
+F 0 "H1" H 4400 7421 50  0000 L CNN
+F 1 "MountingHole" H 4400 7330 50  0000 L CNN
+F 2 "MountingHole:MountingHole_2.1mm" H 4300 7375 50  0001 C CNN
+F 3 "~" H 4300 7375 50  0001 C CNN
+	1    4300 7375
+	1    0    0    -1
+$EndComp
 $EndSCHEMATC

Commit message: More PCB WIP.
Parts:
- removed U1, U2: OP275, Package_SO:SOIC-8_3.9x4.9mm_P1.27mm, symbol Amplifier_Operational:OP275
- added U1, U2: TLC2722, Package_SO:SOIC-8_3.9x4.9mm_P1.27mm, symbol Amplifier_Operational:LM2904
- H1, H2: footprint MountingHole:MountingHole_2.1mm -> MountingHole:MountingHole_4.3mm_M4
Connections:
- net +5V: now also U1.8 (V+), U2.8 (V+)
- net GND: now also U1.4 (V-), U2.4 (V-)
- net LEDon1: now also XA1.D24; no longer XA1.D23
- net LEDon2: now also XA1.D26; no longer XA1.D24
- net LEDon3: now also XA1.D28; no longer XA1.D25
- net PWMin0: now also XA1.D2 (D2_INT0); no longer XA1.D46
- net PWMin1: now also XA1.D3 (D3_INT1); no longer XA1.D45
- net PWMin2: now also XA1.D4; no longer XA1.D44
- net PWMin3: now also XA1.D5; no longer XA1.D13
- net at R2.2, R3.1: now also U1.3 (+)
- net at Q1.2 (E), R6.2: now also U1.2 (-)
- net at Q1.1 (B): now also U1.1
- net at Q3.2 (E), R11.2: now also U1.6 (-)
- net at Q3.1 (B): now also U1.7
- net at R8.2, R9.1: now also U1.5 (+)
- net at Q7.2 (E), R21.2: now also U2.2 (-)
- net at Q7.1 (B): now also U2.1
- net at R15.2, R17.1: now also U2.3 (+)
- net at Q5.2 (E), R20.2: now also U2.6 (-)
- net at Q5.1 (B): now also U2.7
- net at R14.2, R16.1: now also U2.5 (+)
Changed lines of the file:
@@
-$EndComp
-$Comp
-L Amplifier_Operational:OP275 U1
-U 1 1 5FF96DDF
-P 2625 1500
-F 0 "U1" H 2625 1867 50  0000 C CNN
-F 1 "OP275" H 2625 1776 50  0000 C CNN
-F 2 "Package_SO:SOIC-8_3.9x4.9mm_P1.27mm" H 2625 1500 50  0001 C CNN
-F 3 "https://www.analog.com/media/en/technical-documentation/data-sheets/OP275.pdf" H 2625 1500 50  0001 C CNN
-	1    2625 1500
-	1    0    0    -1
-$EndComp
-$Comp
-L Amplifier_Operational:OP275 U1
-U 2 1 5FFA949E
-P 6225 1500
-F 0 "U1" H 6225 1867 50  0000 C CNN
-F 1 "OP275" H 6225 1776 50  0000 C CNN
-F 2 "Package_SO:SOIC-8_3.9x4.9mm_P1.27mm" H 6225 1500 50  0001 C CNN
-F 3 "https://www.analog.com/media/en/technical-documentation/data-sheets/OP275.pdf" H 6225 1500 50  0001 C CNN
-	2    6225 1500
-	1    0    0    -1
-$EndComp
-$Comp
-L Amplifier_Operational:OP275 U2
-U 1 1 5FFAB683
-P 9550 1600
-F 0 "U2" H 9550 1967 50  0000 C CNN
-F 1 "OP275" H 9550 1876 50  0000 C CNN
-F 2 "Package_SO:SOIC-8_3.9x4.9mm_P1.27mm" H 9550 1600 50  0001 C CNN
-F 3 "https://www.analog.com/media/en/technical-documentation/data-sheets/OP275.pdf" H 9550 1600 50  0001 C CNN
-	1    9550 1600
-	1    0    0    -1
-$EndComp
-$Comp
-L Amplifier_Operational:OP275 U2
-U 2 1 5FFADA40
-P 9525 4350
-F 0 "U2" H 9525 4717 50  0000 C CNN
-F 1 "OP275" H 9525 4626 50  0000 C CNN
-F 2 "Package_SO:SOIC-8_3.9x4.9mm_P1.27mm" H 9525 4350 50  0001 C CNN
-F 3 "https://www.analog.com/media/en/technical-documentation/data-sheets/OP275.pdf" H 9525 4350 50  0001 C CNN
-	2    9525 4350
-	1    0    0    -1
 $EndComp
 $Comp
@@
 Wire Wire Line
 	3000 3725 3050 3725
-Text GLabel 3050 6525 3    50   Input ~ 0
+Text GLabel 6650 6525 3    50   Input ~ 0
 PWMin0
-Text GLabel 3150 6525 3    50   Input ~ 0
+Text GLabel 6550 6525 3    50   Input ~ 0
 PWMin1
-Text GLabel 3250 6525 3    50   Input ~ 0
+Text GLabel 6450 6525 3    50   Input ~ 0
 PWMin2
-Text GLabel 5550 6525 3    50   Input ~ 0
+Text GLabel 6350 6525 3    50   Input ~ 0
 PWMin3
 Text GLabel 5450 6525 3    50   Input ~ 0
 LEDon0
-Text GLabel 5350 6525 3    50   Input ~ 0
+Text GLabel 5250 6525 3    50   Input ~ 0
 LEDon1
-Text GLabel 5250 6525 3    50   Input ~ 0
+Text GLabel 5050 6525 3    50   Input ~ 0
 LEDon2
-Text GLabel 5150 6525 3    50   Input ~ 0
+Text GLabel 4850 6525 3    50   Input ~ 0
 LEDon3
 Text GLabel 5350 3625 1    50   Input ~ 0
@@
 	5350 3725 5350 3625
 Wire Wire Line
-	3050 6525 3050 6325
-Wire Wire Line
-	3150 6525 3150 6325
-Wire Wire Line
-	3250 6525 3250 6325
-Wire Wire Line
-	5150 6525 5150 6325
-Wire Wire Line
-	5250 6525 5250 6325
-Wire Wire Line
-	5350 6525 5350 6325
-Wire Wire Line
 	5450 6525 5450 6325
-Wire Wire Line
-	5550 6525 5550 6325
 $Comp
 L Connector:Conn_01x02_Male J1
@@
 F 0 "H2" H 4650 7421 50  0000 L CNN
 F 1 "MountingHole" H 4650 7330 50  0000 L CNN
-F 2 "MountingHole:MountingHole_2.1mm" H 4550 7375 50  0001 C CNN
+F 2 "MountingHole:MountingHole_4.3mm_M4" H 4550 7375 50  0001 C CNN
 F 3 "~" H 4550 7375 50  0001 C CNN
 	1    4550 7375
@@
 F 0 "H1" H 4400 7421 50  0000 L CNN
 F 1 "MountingHole" H 4400 7330 50  0000 L CNN
-F 2 "MountingHole:MountingHole_2.1mm" H 4300 7375 50  0001 C CNN
+F 2 "MountingHole:MountingHole_4.3mm_M4" H 4300 7375 50  0001 C CNN
 F 3 "~" H 4300 7375 50  0001 C CNN
 	1    4300 7375
 	1    0    0    -1
 $EndComp
+Wire Wire Line
+	6650 6525 6650 6325
+Wire Wire Line
+	6550 6525 6550 6325
+Wire Wire Line
+	5250 6525 5250 6325
+Wire Wire Line
+	5050 6325 5050 6525
+Wire Wire Line
+	4850 6525 4850 6325
+Wire Wire Line
+	6450 6525 6450 6325
+Wire Wire Line
+	6350 6325 6350 6525
+$Comp
+L Amplifier_Operational:LM2904 U1
+U 1 1 600B93BA
+P 2625 1500
+F 0 "U1" H 2625 1867 50  0000 C CNN
+F 1 "TLC2722" H 2625 1776 50  0000 C CNN
+F 2 "Package_SO:SOIC-8_3.9x4.9mm_P1.27mm" H 2625 1500 50  0001 C CNN
+F 3 "http://www.ti.com/lit/ds/symlink/lm358.pdf" H 2625 1500 50  0001 C CNN
+	1    2625 1500
+	1    0    0    -1
+$EndComp
+$Comp
+L Amplifier_Operational:LM2904 U1
+U 2 1 600D1945
+P 6225 1500
+F 0 "U1" H 6225 1867 50  0000 C CNN
+F 1 "TLC2722" H 6225 1776 50  0000 C CNN
+F 2 "Package_SO:SOIC-8_3.9x4.9mm_P1.27mm" H 6225 1500 50  0001 C CNN
+F 3 "http://www.ti.com/lit/ds/symlink/lm358.pdf" H 6225 1500 50  0001 C CNN
+	2    6225 1500
+	1    0    0    -1
+$EndComp
+$Comp
+L Amplifier_Operational:LM2904 U1
+U 3 1 600D5316
+P 1275 2200
+F 0 "U1" H 1233 2246 50  0000 L CNN
+F 1 "TLC2722" H 1233 2155 50  0000 L CNN
+F 2 "Package_SO:SOIC-8_3.9x4.9mm_P1.27mm" H 1275 2200 50  0001 C CNN
+F 3 "http://www.ti.com/lit/ds/symlink/lm358.pdf" H 1275 2200 50  0001 C CNN
+	3    1275 2200
+	1    0    0    -1
+$EndComp
+$Comp
+L Amplifier_Operational:LM2904 U2
+U 1 1 600DA883
+P 9550 1600
+F 0 "U2" H 9550 1967 50  0000 C CNN
+F 1 "TLC2722" H 9550 1876 50  0000 C CNN
+F 2 "Package_SO:SOIC-8_3.9x4.9mm_P1.27mm" H 9550 1600 50  0001 C CNN
+F 3 "http://www.ti.com/lit/ds/symlink/lm358.pdf" H 9550 1600 50  0001 C CNN
+	1    9550 1600
+	1    0    0    -1
+$EndComp
+$Comp
+L Amplifier_Operational:LM2904 U2
+U 2 1 600DD659
+P 9525 4350
+F 0 "U2" H 9525 4717 50  0000 C CNN
+F 1 "TLC2722" H 9525 4626 50  0000 C CNN
+F 2 "Package_SO:SOIC-8_3.9x4.9mm_P1.27mm" H 9525 4350 50  0001 C CNN
+F 3 "http://www.ti.com/lit/ds/symlink/lm358.pdf" H 9525 4350 50  0001 C CNN
+	2    9525 4350
+	1    0    0    -1
+$EndComp
+$Comp
+L Amplifier_Operational:LM2904 U2
+U 3 1 600DFE65
+P 8250 2225
+F 0 "U2" H 8208 2271 50  0000 L CNN
+F 1 "TLC2722" H 8208 2180 50  0000 L CNN
+F 2 "Package_SO:SOIC-8_3.9x4.9mm_P1.27mm" H 8250 2225 50  0001 C CNN
+F 3 "http://www.ti.com/lit/ds/symlink/lm358.pdf" H 8250 2225 50  0001 C CNN
+	3    8250 2225
+	1    0    0    -1
+$EndComp
+$Comp
+L power:+5V #PWR0103
+U 1 1 600EF611
+P 1175 1900
+F 0 "#PWR0103" H 1175 1750 50  0001 C CNN
+F 1 "+5V" H 1190 2073 50  0000 C CNN
+F 2 "" H 1175 1900 50  0001 C CNN
+F 3 "" H 1175 1900 50  0001 C CNN
+	1    1175 1900
+	1    0    0    -1
+$EndComp
+$Comp
+L power:GND #PWR0104
+U 1 1 600F06EC
+P 1175 2500
+F 0 "#PWR0104" H 1175 2250 50  0001 C CNN
+F 1 "GND" H 1180 2327 50  0000 C CNN
+F 2 "" H 1175 2500 50  0001 C CNN
+F 3 "" H 1175 2500 50  0001 C CNN
+	1    1175 2500
+	1    0    0    -1
+$EndComp
+$Comp
+L power:GND #PWR0105
+U 1 1 600F153A
+P 8150 2525
+F 0 "#PWR0105" H 8150 2275 50  0001 C CNN
+F 1 "GND" H 8155 2352 50  0000 C CNN
+F 2 "" H 8150 2525 50  0001 C CNN
+F 3 "" H 8150 2525 50  0001 C CNN
+	1    8150 2525
+	1    0    0    -1
+$EndComp
+$Comp
+L power:+5V #PWR0106
+U 1 1 600F249E
+P 8150 1925
+F 0 "#PWR0106" H 8150 1775 50  0001 C CNN
+F 1 "+5V" H 8165 2098 50  0000 C CNN
+F 2 "" H 8150 1925 50  0001 C CNN
+F 3 "" H 8150 1925 50  0001 C CNN
+	1    8150 1925
+	1    0    0    -1
+$EndComp

Commit message: More PCB WIP...
Parts:
- removed H1, H2: MountingHole, MountingHole:MountingHole_4.3mm_M4, symbol Mechanical:MountingHole
- removed XA1: Arduino_Mega2560_Shield, arduino:Arduino_Mega2560_Shield, symbol arduino:Arduino_Mega2560_Shield
- added XA1: Arduino_Mega2560_Shield, reprapltd-kicad:Arduino_Mega2560_Shield, symbol reprapltd-kicad:Arduino_Mega2560_Shield
Connections:
- net +5V: now also XA1.5V1 (5V)
- net GND: now also XA1.GND3 (GND)
- net LEDon0: now also XA1.D24
- net LEDon1: now also XA1.D26
- net LEDon2: now also XA1.D28
- net LEDon3: now also XA1.D30
- net PWMin0: now also XA1.D10
- net PWMin1: now also XA1.D11
- net PWMin2: now also XA1.D12
- net PWMin3: now also XA1.D13
- net photoC: now also XA1.A0
- net at R3.1, U1.3 (+): now also R14.2; no longer R2.2
- net at Q3.2 (E), R11.2: now also U2.2 (-); no longer U1.6 (-)
- net at Q3.1 (B): now also U2.1; no longer U1.7
- net at R8.2, R9.1: now also U2.3 (+); no longer U1.5 (+)
- net at Q7.2 (E), R21.2: now also U1.6 (-); no longer U2.2 (-)
- net at Q7.1 (B): now also U1.7; no longer U2.1
- net at R15.2, R17.1: now also U1.5 (+); no longer U2.3 (+)
- net at R16.1, U2.5 (+): now also R2.2; no longer R14.2
- new net: XA1.5V3 (5V), XA1.5V4 (5V)
- new net: XA1.GND5 (GND), XA1.GND6 (GND)
Other:
- moved on the sheet: C1, C4, R1, R12, R14, R2, U1B, U2A

Commit message: First finished PCB.
Connections:
- net LEDon0: now also XA1.D46; no longer XA1.D24
- net LEDon1: now also XA1.D48; no longer XA1.D26
- net LEDon2: now also XA1.D50; no longer XA1.D28
- net LEDon3: now also XA1.D52; no longer XA1.D30
Changed lines of the file:
@@
 Wire Wire Line
 	3000 3600 3000 3725
-Text GLabel 5250 6525 3    50   Input ~ 0
+Text GLabel 3050 6525 3    50   Input ~ 0
 LEDon0
-Text GLabel 5050 6525 3    50   Input ~ 0
+Text GLabel 2850 6525 3    50   Input ~ 0
 LEDon1
-Text GLabel 4850 6525 3    50   Input ~ 0
+Text GLabel 2650 6525 3    50   Input ~ 0
 LEDon2
-Text GLabel 4650 6525 3    50   Input ~ 0
+Text GLabel 2450 6525 3    50   Input ~ 0
 LEDon3
 Text GLabel 5350 3625 1    50   Input ~ 0
@@
 	5350 3725 5350 3625
 Wire Wire Line
-	5250 6525 5250 6325
+	3050 6525 3050 6325
 $Comp
 L Connector:Conn_01x02_Male J1
@@
 Connection ~ 1625 6775
 Wire Wire Line
-	5050 6525 5050 6325
+	2850 6525 2850 6325
 Wire Wire Line
-	4850 6325 4850 6525
+	2650 6325 2650 6525
 Wire Wire Line
-	4650 6525 4650 6325
+	2450 6525 2450 6325
 $Comp
 L Amplifier_Operational:LM2904 U1

Commit message: PCB GERBERS.
Connections:
- net +5V: now also XA1.5V3 (5V), XA1.5V4 (5V)
- net GND: now also XA1.GND1 (GND), XA1.GND2 (GND), XA1.GND5 (GND), XA1.GND6 (GND)
Changed lines of the file:
@@
 Connection ~ 2200 1400
 Connection ~ 9100 4250
+Wire Wire Line
+	2950 3725 3000 3725
+Connection ~ 2950 3725
+Connection ~ 3000 3725
+Wire Wire Line
+	3050 3725 3150 3725
+Connection ~ 3050 3725
+Wire Wire Line
+	3150 3725 3250 3725
+Connection ~ 3150 3725
+Wire Wire Line
+	2600 3725 2550 3725
+Connection ~ 2600 3725
+Connection ~ 2550 3725
 $EndSCHEMATC

Commit message: Now with better resistance values...
Parts:
- R11, R20, R21, R6: value 100R -> 470R
- R5: value 3K3 -> 560R
Other:
- note added: "Maybe make 120K 100K on op amp input."
Changed lines of the file:
@@
 P 3375 1975
 F 0 "R6" H 3305 1929 50  0000 R CNN
-F 1 "100R" H 3305 2020 50  0000 R CNN
+F 1 "470R" H 3305 2020 50  0000 R CNN
 F 2 "Resistor_SMD:R_0805_2012Metric" V 3305 1975 50  0001 C CNN
 F 3 "~" H 3375 1975 50  0001 C CNN
@@
 P 6975 1975
 F 0 "R11" H 6905 1929 50  0000 R CNN
-F 1 "100R" H 6905 2020 50  0000 R CNN
+F 1 "470R" H 6905 2020 50  0000 R CNN
 F 2 "Resistor_SMD:R_0805_2012Metric" V 6905 1975 50  0001 C CNN
 F 3 "~" H 6975 1975 50  0001 C CNN
@@
 P 10300 2075
 F 0 "R21" H 10230 2029 50  0000 R CNN
-F 1 "100R" H 10230 2120 50  0000 R CNN
+F 1 "470R" H 10230 2120 50  0000 R CNN
 F 2 "Resistor_SMD:R_0805_2012Metric" V 10230 2075 50  0001 C CNN
 F 3 "~" H 10300 2075 50  0001 C CNN
@@
 P 10275 4825
 F 0 "R20" H 10205 4779 50  0000 R CNN
-F 1 "100R" H 10205 4870 50  0000 R CNN
+F 1 "470R" H 10205 4870 50  0000 R CNN
 F 2 "Resistor_SMD:R_0805_2012Metric" V 10205 4825 50  0001 C CNN
 F 3 "~" H 10275 4825 50  0001 C CNN
@@
 P 1625 6475
 F 0 "R5" H 1555 6429 50  0000 R CNN
-F 1 "3K3" H 1555 6520 50  0000 R CNN
+F 1 "560R" H 1555 6520 50  0000 R CNN
 F 2 "Resistor_SMD:R_0805_2012Metric" V 1555 6475 50  0001 C CNN
 F 3 "~" H 1625 6475 50  0001 C CNN
@@
 Connection ~ 2600 3725
 Connection ~ 2550 3725
+Text Notes 3500 675  0    50   ~ 0
+Maybe make 120K 100K on op amp input.
 $EndSCHEMATC
