File: Electronics/LED-shield/LED-shield.kicad_pcb (KiCad board)
At the start: 2 copper layers, 68.6 x 53.3 mm, 31 parts, among them U1 PCA9622

Commit message: WIP on pure electronic version
Other:
- net class Default removed
