File: Electronics/one-synapse-electronic/one-synapse-electronic/one-synapse-electronic.kicad_pcb (KiCad board)
At the start: 2 copper layers, 92.2 x 72.5 mm, 137 parts, among them J1 prg-err, J10 comb, J2 Axon, J3 Axon, J4 PWM-in, J5 PWM-out, J6 pwr, J7 synapses, J9 sel, Q17 BS170F, Q18 BS170F, Q19 BS170F, Q20 BS170F, Q21 BS170F, Q22 BS170F, Q23 BS170F, Q24 BS170F, Q25 BS170F, Q26 BS170F, Q27 BS170F, Q28 BS170F, Q29 BS170F, Q30 BS170F, Q31 BS170F, Q32 BS170F, U1 TLC5940PWP, U2 MCP6004, U3 MCP6004, U4 MCP6004, U5 MCP6004, U6 MCP6004

Commit message: 2nd final PCB design...
Parts:
- J5: moved to B.Cu
- moved J5 15.2 mm to (141.2, 143.9)
Connections:
- H1 pad : (no net) -> GND
- H2 pad : (no net) -> GND
- H3 pad : (no net) -> GND
- H4 pad : (no net) -> GND
Routing:
- net GSCLK: track 171.4 -> 187.7 mm
- net XLAT: track 167.2 -> 176.9 mm
- net Net-(J9-Pin_2): track 62.5 -> 54.8 mm, vias 2 -> 3
- net Vcc: track 309.8 -> 316.5 mm
- net SCLK: track 167.5 -> 162.8 mm, vias 0 -> 1
- net BLANK: track 163.5 -> 167.4 mm
- net Sout: track 170.8 -> 170.1 mm
Other:
- board text added: "+"
- board text added: "+/-"
- board text added: "+5V"
- board text added: "-"
- board text added: "Analogue Artificial Neural Network Synapse RepRap Ltd reprapltd.com Licence: GPL Design: Adrian Bowyer"
- board text added: "BLANK"
- board text added: "Comp"
- board text added: "GND"
- board text added: "GSCLK"
- board text added: "INPUTS"
- board text added: "OUTPUT x 16"
- board text added: "SCLK"
- board text added: "Sin"
- board text added: "Sout"
- board text added: "VPRG"
- board text added: "XERR"
- board text added: "XLAT"
- board text added: "this"
