File: Electronics/Diagrams/crosspoint/axon-synapse-conn.kicad_sch (KiCad schematic)
At the start: 16 parts

Commit message: Add images from svgs
Parts:
- removed R0m, Rqm: ~, symbol Switch:SW_SPST
- added G0, Gn, R0m2, Rqm2, X0m2, Xnm2: ~, symbol Switch:SW_SPST
- added R1: 100K, symbol Device:R
- renumbered X0m to V0, Xnm to Vn
Connections:
- net at V0.1 (A), Vn.1 (A): now also R1.1
- net at Dn0.2 (B), Dnp.2 (B), Vn.2 (B)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: now also Gn.2 (B), Xnm2.2 (B)
- net at D00.2 (B), D0p.2 (B), V0.2 (B)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: now also G0.2 (B), X0m2.2 (B)
- net at DR00.2 (B), DR0p.2 (B), R00.2 (B): now also R0m2.2 (B)
- net at DRq0.2 (B), DRqp.2 (B), Rq0.2 (B): now also Rqm2.2 (B)
- new net: R0m2.1 (A), Rqm2.1 (A), X0m2.1 (A), Xnm2.1 (A)
- new net GNDREF: G0.1 (A), Gn.1 (A)
- new net VDD: R1.2
