File: Electronics/Diagrams/crosspoint/synapse-axon-conn.kicad_sch (KiCad schematic)
At the start: 16 parts, among them U1 L272, U2 L272, U3 L272, U4 L272

Commit message: Add images from svgs
Changed lines of the file:
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@@
     )
     (property "Value" "100K" (at 57.785 86.36 90)
-      (effects (font (size 1.27 1.27)))
+      (effects (font (size 1.27 1.27)) hide)
     )
     (property "Footprint" "" (at 57.785 91.948 90)
@@
     )
     (property "Value" "100K" (at 58.42 26.67 90)
-      (effects (font (size 1.27 1.27)))
+      (effects (font (size 1.27 1.27)) hide)
     )
     (property "Footprint" "" (at 58.42 32.258 90)
