File: Electronics/Crosspoint-AANN/crosspoint-switches/crosspoint-switches.kicad_sch (KiCad schematic)
At the start: 4 parts, among them J1 Conn_02x03_Counter_Clockwise, U2 74LVC1G175

Commit message: PCB WIP
Parts:
- added C2: 0.1u, Capacitor_SMD:C_0805_2012Metric, symbol Device:C
- added J2, J4: Conn_01x16_Pin, Connector_PinSocket_1.27mm:PinSocket_1x16_P1.27mm_Vertical, symbol Connector:Conn_01x16_Pin
- added J3, J5: Conn_01x16_Socket, Connector_PinSocket_1.27mm:PinSocket_1x16_P1.27mm_Vertical, symbol Connector:Conn_01x16_Socket
- C1: value 1u -> 4u7
- J1: footprint (none) -> Connector_PinSocket_1.27mm:PinSocket_2x03_P1.27mm_Vertical
- U1: value ~ -> ADG2188; footprint (none) -> reprapltd-kicad:QFN50P500X500X100-33N
Connections:
- net +5V: now also C2.1, J2.7 (Pin_7), J3.7 (Pin_7), J4.7 (Pin_7), J5.7 (Pin_7)
- net CROSS-RST: now also J2.2 (Pin_2), J3.2 (Pin_2), J4.2 (Pin_2), J5.2 (Pin_2)
- net DLQR: now also J2.1 (Pin_1)
- net GND: now also C2.2, J2.16 (Pin_16), J3.16 (Pin_16), J4.16 (Pin_16), J5.16 (Pin_16)
- net QLDR: now also J3.1 (Pin_1)
- net SCL: now also J2.4 (Pin_4), J3.4 (Pin_4), J4.4 (Pin_4), J5.4 (Pin_4)
- net SDA: now also J2.3 (Pin_3), J3.3 (Pin_3), J4.3 (Pin_3), J5.3 (Pin_3)
- net SHIFT-CLK: now also J2.6 (Pin_6), J3.6 (Pin_6), J4.6 (Pin_6), J5.6 (Pin_6)
- net SHIFT-RST: now also J2.5 (Pin_5), J3.5 (Pin_5), J4.5 (Pin_5), J5.5 (Pin_5)
- net X0: now also J2.15 (Pin_15), J3.15 (Pin_15)
- net X1: now also J2.14 (Pin_14), J3.14 (Pin_14)
- net X2: now also J2.13 (Pin_13), J3.13 (Pin_13)
- net X3: now also J2.12 (Pin_12), J3.12 (Pin_12)
- net X4: now also J2.11 (Pin_11), J3.11 (Pin_11)
- net X5: now also J2.10 (Pin_10), J3.10 (Pin_10)
- net X6: now also J2.9 (Pin_9), J3.9 (Pin_9)
- net X7: now also J2.8 (Pin_8), J3.8 (Pin_8)
- net Y0: now also J4.15 (Pin_15), J5.15 (Pin_15)
- net Y1: now also J4.14 (Pin_14), J5.14 (Pin_14)
- net Y2: now also J4.13 (Pin_13), J5.13 (Pin_13)
- net Y3: now also J4.12 (Pin_12), J5.12 (Pin_12)
- net Y4: now also J4.11 (Pin_11), J5.11 (Pin_11)
- net Y5: now also J4.10 (Pin_10), J5.10 (Pin_10)
- net Y6: now also J4.9 (Pin_9), J5.9 (Pin_9)
- net Y7: now also J4.8 (Pin_8), J5.8 (Pin_8)
- net D: no longer names the net of J1.2 (Pin_2), U2.3 (D)
- net Q: no longer names the net of J1.5 (Pin_5), U1.28 (A0), U2.4 (Q)
Other:
- moved on the sheet: C1, J1, U1, U2

Commit message: PCB WIP
Parts:
- removed J1: Conn_02x03_Counter_Clockwise, Connector_PinSocket_1.27mm:PinSocket_2x03_P1.27mm_Vertical, symbol Connector_Generic:Conn_02x03_Counter_Clockwise
- added J6: Conn_02x03_Odd_Even, Connector_PinSocket_1.27mm:PinSocket_2x03_P1.27mm_Vertical, symbol Connector_Generic:Conn_02x03_Odd_Even
Connections:
- net DLQR: now also J6.1 (Pin_1), J6.6 (Pin_6)
- net QLDR: now also J6.2 (Pin_2), J6.5 (Pin_5)
- net at U1.28 (A0), U2.4 (Q): now also J6.4 (Pin_4)
- net at U2.3 (D): now also J6.3 (Pin_3)
Changed lines of the file:
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@@
+    )
+  )
+  (symbol (lib_id "Connector_Generic:Conn_02x03_Odd_Even") (at 62.23 23.495 0) (unit 1)
+    (in_bom yes) (on_board yes) (dnp no) (fields_autoplaced)
+    (property "Reference" "J6" (at 63.5 14.605 0)
+      (effects (font (size 1.27 1.27)))
+    )
+    (property "Value" "Conn_02x03_Odd_Even" (at 63.5 17.145 0)
+      (effects (font (size 1.27 1.27)))
+    )
+    (property "Footprint" "Connector_PinSocket_1.27mm:PinSocket_2x03_P1.27mm_Vertical" (at 62.23 23.495 0)
+      (effects (font (size 1.27 1.27)) hide)
+    )
+    (property "Datasheet" "~" (at 62.23 23.495 0)
+      (effects (font (size 1.27 1.27)) hide)
+    )
+    (pin "4")
+    (pin "2")
+    (pin "1")
+    (pin "3")
+    (pin "6")
+    (pin "5")
+    (instances
+      (project "crosspoint-switches"
+        (path "/7befdfce-0150-4a1c-9211-f99285b6f61d"
+          (reference "J6") (unit 1)
+        )
+      )
     )
   )
@@
         )
       )
-    )
-  )
-  (symbol (lib_id "Connector_Generic:Conn_02x03_Counter_Clockwise") (at 62.23 23.495 0) (unit 1)
-    (in_bom yes) (on_board yes) (dnp no)
-    (property "Reference" "J1" (at 63.5 17.78 0)
-      (effects (font (size 1.27 1.27)))
-    )
-    (property "Value" "Conn_02x03_Counter_Clockwise" (at 63.5 17.145 0)
-      (effects (font (size 1.27 1.27)) hide)
-    )
-    (property "Footprint" "Connector_PinSocket_1.27mm:PinSocket_2x03_P1.27mm_Vertical" (at 62.23 23.495 0)
-      (effects (font (size 1.27 1.27)) hide)
-    )
-    (property "Datasheet" "~" (at 62.23 23.495 0)
-      (effects (font (size 1.27 1.27)) hide)
-    )
-    (pin "4")
-    (pin "1")
-    (pin "6")
-    (pin "2")
-    (pin "3")
-    (pin "5")
-    (instances
-      (project "crosspoint-switches"
-        (path "/7befdfce-0150-4a1c-9211-f99285b6f61d"
-          (reference "J1") (unit 1)
-        )
-      )

Commit message: PCB WIP
Parts:
- added C3: 0.1u, Capacitor_SMD:C_0805_2012Metric, symbol Device:C
Connections:
- net +5V: now also C3.1
- net GND: now also U1.33 (EPAD), C3.2; no longer U1.32 (GND), U1.pad (EPAD)
Changed lines of the file:
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@@
   (junction (at 179.705 85.09) (diameter 0) (color 0 0 0 0)
   )
-  (junction (at 99.695 51.435) (diameter 0) (color 0 0 0 0)
-  )
   (wire (pts (xy 38.735 133.35) (xy 59.055 133.35))
     (stroke (width 0) (type default))
@@
     (stroke (width 0) (type default))
   )
+  (wire (pts (xy 99.695 48.895) (xy 99.695 48.895))
+    (stroke (width 0) (type default))
+  )
+  (wire (pts (xy 113.665 71.755) (xy 113.665 80.01))
+    (stroke (width 0) (type default))
+  )
+  (wire (pts (xy 41.91 146.05) (xy 41.91 147.32))
+    (stroke (width 0) (type default))
+  )
+  (wire (pts (xy 210.185 129.54) (xy 210.185 126.365))
+    (stroke (width 0) (type default))
+  )
+  (wire (pts (xy 72.39 20.955) (xy 72.39 30.48))
+    (stroke (width 0) (type default))
+  )
+  (wire (pts (xy 110.49 36.195) (xy 111.76 36.195))
+    (stroke (width 0) (type default))
+  )
+  (wire (pts (xy 93.98 53.975) (xy 99.695 53.975))
+    (stroke (width 0) (type default))
+  )
+  (wire (pts (xy 48.26 23.495) (xy 57.15 23.495))
+    (stroke (width 0) (type default))
+  )
   (wire (pts (xy 99.695 51.435) (xy 99.695 53.975))
     (stroke (width 0) (type default))
   )
-  (wire (pts (xy 113.665 71.755) (xy 113.665 80.01))
-    (stroke (width 0) (type default))
-  )
-  (wire (pts (xy 41.91 146.05) (xy 41.91 147.32))
-    (stroke (width 0) (type default))
-  )
-  (wire (pts (xy 210.185 129.54) (xy 210.185 126.365))
-    (stroke (width 0) (type default))
-  )
-  (wire (pts (xy 72.39 20.955) (xy 72.39 30.48))
-    (stroke (width 0) (type default))
-  )
-  (wire (pts (xy 110.49 36.195) (xy 111.76 36.195))
-    (stroke (width 0) (type default))
-  )
-  (wire (pts (xy 93.98 53.975) (xy 99.695 53.975))
-    (stroke (width 0) (type default))
-  )
-  (wire (pts (xy 48.26 23.495) (xy 57.15 23.495))
-    (stroke (width 0) (type default))
-  )
   (wire (pts (xy 38.735 146.05) (xy 41.91 146.05))
     (stroke (width 0) (type default))
@@
     (stroke (width 0) (type default))
   )
-  (wire (pts (xy 99.695 48.895) (xy 99.695 51.435))
-    (stroke (width 0) (type default))
-  )
   (wire (pts (xy 177.165 129.54) (xy 177.165 81.28))
     (stroke (width 0) (type default))
@@
         (path "/7befdfce-0150-4a1c-9211-f99285b6f61d"
           (reference "#PWR06") (unit 1)
+        )
+      )
+    )
+  )
+  (symbol (lib_id "Device:C") (at 24.765 86.995 0) (unit 1)
+    (in_bom yes) (on_board yes) (dnp no) (fields_autoplaced)
+    (property "Reference" "C3" (at 28.575 85.725 0)
+      (effects (font (size 1.27 1.27)) (justify left))
+    )
+    (property "Value" "0.1u" (at 28.575 88.265 0)
+      (effects (font (size 1.27 1.27)) (justify left))
+    )
+    (property "Footprint" "Capacitor_SMD:C_0805_2012Metric" (at 25.7302 90.805 0)
+      (effects (font (size 1.27 1.27)) hide)
+    )
+    (property "Datasheet" "~" (at 24.765 86.995 0)
+      (effects (font (size 1.27 1.27)) hide)
+    )
+    (pin "1")
+    (pin "2")
+    (instances
+      (project "crosspoint-switches"
+        (path "/7befdfce-0150-4a1c-9211-f99285b6f61d"
+          (reference "C3") (unit 1)
         )
       )
@@
     )
   )
+  (symbol (lib_id "power:GND") (at 24.765 90.805 0) (unit 1)
+    (in_bom yes) (on_board yes) (dnp no) (fields_autoplaced)
+    (property "Reference" "#PWR014" (at 24.765 97.155 0)
+      (effects (font (size 1.27 1.27)) hide)
+    )
+    (property "Value" "GND" (at 24.765 95.25 0)
+      (effects (font (size 1.27 1.27)))
+    )
+    (property "Footprint" "" (at 24.765 90.805 0)
+      (effects (font (size 1.27 1.27)) hide)
+    )
+    (property "Datasheet" "" (at 24.765 90.805 0)
+      (effects (font (size 1.27 1.27)) hide)
+    )
+    (pin "1")
+    (instances
+      (project "crosspoint-switches"
+        (path "/7befdfce-0150-4a1c-9211-f99285b6f61d"
+          (reference "#PWR014") (unit 1)
+        )
+      )
+    )
+  )
   (symbol (lib_id "power:GND") (at 64.77 64.77 0) (unit 1)
     (in_bom yes) (on_board yes) (dnp no) (fields_autoplaced)
@@
         (path "/7befdfce-0150-4a1c-9211-f99285b6f61d"
           (reference "#PWR04") (unit 1)
-        )
-      )
-    )
-  )
-  (symbol (lib_id "reprapltd-kicad:ADG2188") (at 114.935 53.34 0) (unit 1)
-    (in_bom yes) (on_board yes) (dnp no)
-    (property "Reference" "U1" (at 113.665 53.34 0)
-      (effects (font (size 1.27 1.27)) (justify left))
-    )
-    (property "Value" "ADG2188" (at 114.935 56.515 0)
-      (effects (font (size 1.27 1.27)))
-    )
-    (property "Footprint" "reprapltd-kicad:QFN50P500X500X100-33N" (at 114.935 56.515 0)
-      (effects (font (size 1.27 1.27)) hide)
-    )
-    (property "Datasheet" "" (at 114.935 56.515 0)
-      (effects (font (size 1.27 1.27)) hide)
-    )
-    (pin "27")
-    (pin "pad")
-    (pin "9")
-    (pin "8")
-    (pin "17")
-    (pin "15")
-    (pin "4")
-    (pin "26")
-    (pin "18")
-    (pin "24")
-    (pin "25")
-    (pin "29")
-    (pin "12")
-    (pin "16")
-    (pin "14")
-    (pin "30")
-    (pin "13")
-    (pin "3")
-    (pin "6")
-    (pin "5")
-    (pin "7")
-    (pin "28")
-    (pin "11")
-    (pin "32")
-    (pin "10")
-    (pin "1")
-    (pin "31")
-    (instances
-      (project "crosspoint-switches"
-        (path "/7befdfce-0150-4a1c-9211-f99285b6f61d"
-          (reference "U1") (unit 1)
         )
       )
@@
         (path "/7befdfce-0150-4a1c-9211-f99285b6f61d"
           (reference "#PWR011") (unit 1)
+        )
+      )
+    )
+  )
+  (symbol (lib_id "power:+5V") (at 24.765 83.185 0) (unit 1)
+    (in_bom yes) (on_board yes) (dnp no) (fields_autoplaced)
+    (property "Reference" "#PWR013" (at 24.765 86.995 0)
+      (effects (font (size 1.27 1.27)) hide)
+    )
+    (property "Value" "+5V" (at 24.765 78.74 0)
+      (effects (font (size 1.27 1.27)))
+    )
+    (property "Footprint" "" (at 24.765 83.185 0)
+      (effects (font (size 1.27 1.27)) hide)
+    )
+    (property "Datasheet" "" (at 24.765 83.185 0)
+      (effects (font (size 1.27 1.27)) hide)
+    )
+    (pin "1")
+    (instances
+      (project "crosspoint-switches"
+        (path "/7befdfce-0150-4a1c-9211-f99285b6f61d"
+          (reference "#PWR013") (unit 1)
         )
       )
@@
         )
       )
+    )
+  )
+  (symbol (lib_id "reprapltd-kicad:ADG2188") (at 114.935 53.34 0) (unit 1)
+    (in_bom yes) (on_board yes) (dnp no) (fields_autoplaced)
+    (property "Reference" "U1" (at 117.7641 36.83 0)
+      (effects (font (size 1.27 1.27)) (justify left))
+    )
+    (property "Value" "ADG2188" (at 114.935 56.515 0)
+      (effects (font (size 1.27 1.27)))
+    )
+    (property "Footprint" "reprapltd-kicad:QFN50P500X500X100-33N" (at 114.935 56.515 0)
+      (effects (font (size 1.27 1.27)) hide)
+    )
+    (property "Datasheet" "" (at 114.935 56.515 0)
+      (effects (font (size 1.27 1.27)) hide)
+    )
+    (pin "5")
+    (pin "17")
+    (pin "6")
+    (pin "3")
+    (pin "28")
+    (pin "24")
+    (pin "7")
+    (pin "31")
+    (pin "30")
+    (pin "29")
+    (pin "4")
+    (pin "8")
+    (pin "32")
+    (pin "25")
+    (pin "9")
+    (pin "18")
+    (pin "33")
+    (pin "26")
+    (pin "10")
+    (pin "13")
+    (pin "12")
+    (pin "1")
+    (pin "27")
+    (pin "16")
+    (pin "11")
+    (pin "15")
+    (pin "14")
+    (instances
+      (project "crosspoint-switches"
+        (path "/7befdfce-0150-4a1c-9211-f99285b6f61d"
+          (reference "U1") (unit 1)
+        )
+      )

Commit message: PCB WIP
Parts:
- added H1, H2, H3, H4: MountingHole_Pad, MountingHole:MountingHole_2.2mm_M2_DIN965_Pad, symbol Mechanical:MountingHole_Pad
Connections:
- net +5V: now also J2.10 (Pin_10), J3.10 (Pin_10); no longer J2.7 (Pin_7), J3.7 (Pin_7)
- net CROSS-RST: now also J2.15 (Pin_15), J3.15 (Pin_15); no longer J2.2 (Pin_2), J3.2 (Pin_2)
- net DLQR: now also J2.16 (Pin_16); no longer J2.1 (Pin_1)
- net GND: now also J2.1 (Pin_1), J3.1 (Pin_1), H1.1, H2.1, H3.1, H4.1; no longer J2.16 (Pin_16), J3.16 (Pin_16)
- net QLDR: now also J3.16 (Pin_16); no longer J3.1 (Pin_1)
- net SCL: now also J2.13 (Pin_13), J3.13 (Pin_13); no longer J2.4 (Pin_4), J3.4 (Pin_4)
- net SDA: now also J2.14 (Pin_14), J3.14 (Pin_14); no longer J2.3 (Pin_3), J3.3 (Pin_3)
- net SHIFT-CLK: now also J2.11 (Pin_11), J3.11 (Pin_11); no longer J2.6 (Pin_6), J3.6 (Pin_6)
- net SHIFT-RST: now also J2.12 (Pin_12), J3.12 (Pin_12); no longer J2.5 (Pin_5), J3.5 (Pin_5)
- net X0: now also J2.9 (Pin_9), J3.9 (Pin_9); no longer J2.15 (Pin_15), J3.15 (Pin_15)
- net X1: now also J2.8 (Pin_8), J3.8 (Pin_8); no longer J2.14 (Pin_14), J3.14 (Pin_14)
- net X2: now also J2.7 (Pin_7), J3.7 (Pin_7); no longer J2.13 (Pin_13), J3.13 (Pin_13)
- net X3: now also J2.6 (Pin_6), J3.6 (Pin_6); no longer J2.12 (Pin_12), J3.12 (Pin_12)
- net X4: now also J2.5 (Pin_5), J3.5 (Pin_5); no longer J2.11 (Pin_11), J3.11 (Pin_11)
- net X5: now also J2.4 (Pin_4), J3.4 (Pin_4); no longer J2.10 (Pin_10), J3.10 (Pin_10)
- net X6: now also J2.3 (Pin_3), J3.3 (Pin_3); no longer J2.9 (Pin_9), J3.9 (Pin_9)
- net X7: now also J2.2 (Pin_2), J3.2 (Pin_2); no longer J2.8 (Pin_8), J3.8 (Pin_8)

Commit message: PCB WIP
Connections:
- net GND: now also U1.32 (GND)
Changed lines of the file:
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@@
   (junction (at 111.76 36.195) (diameter 0) (color 0 0 0 0)
   )
+  (junction (at 93.98 48.895) (diameter 0) (color 0 0 0 0)
+  )
   (junction (at 189.865 101.6) (diameter 0) (color 0 0 0 0)
   )
@@
     (stroke (width 0) (type default))
   )
-  (wire (pts (xy 93.98 32.385) (xy 93.98 53.975))
+  (wire (pts (xy 93.98 32.385) (xy 93.98 48.895))
     (stroke (width 0) (type default))
   )
@@
     (stroke (width 0) (type default))
   )
+  (wire (pts (xy 93.98 48.895) (xy 93.98 53.975))
+    (stroke (width 0) (type default))
+  )
   (wire (pts (xy 71.12 104.775) (xy 71.12 123.19))
     (stroke (width 0) (type default))
@@
     (stroke (width 0) (type default))
   )
+  (wire (pts (xy 93.98 48.895) (xy 99.695 48.895))
+    (stroke (width 0) (type default))
+  )

Commit message: First crosspoint block PCB design.
Parts:
- added D1, D2: LED R, LED_SMD:LED_0805_2012Metric, symbol Device:LED
- added D3, D4: LED G, LED_SMD:LED_0805_2012Metric, symbol Device:LED
- added R1, R2: R470, Resistor_SMD:R_0805_2012Metric, symbol Device:R
Connections:
- net +5V: now also R1.2
- net GND: now also D2.1 (K), D4.1 (K)
- net at J6.4 (Pin_4), U1.28 (A0), U2.4 (Q): now also R2.2
- new net: D3.1 (K), D4.2 (A)
- new net: D1.2 (A), R1.1
- new net: D3.2 (A), R2.1
- new net: D1.1 (K), D2.2 (A)
Other:
- moved on the sheet: C1, C2, C3
